File: EDID_EMULATION.kicad_sch (KiCad schematic)
At the start: 8 parts, among them U2 M24C02-RMN, U4 TMUX1574DYY, U5 TMUX1574DYY

Commit message: Created Branch and Made Changes
Fixed I2C going into Mux shorting the 3V3 side and 5V side due to nets being the same names. Added grounding to HDMI Out connector. Fixed footprint for TS3DV642A0RUAR to use KiCAD default library footprint with EasyEDA 3D model.
Connections:
- net uC_I2C1_SCL renamed 5V_uC_I2C1_SCL
- net uC_I2C1_SDA renamed 5V_uC_I2C1_SDA
Changed lines of the file:
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@@
 	(wire
 		(pts
-			(xy 153.67 48.26) (xy 170.18 48.26)
-		)
-		(stroke
-			(width 0)
-			(type default)
-		)
-	)
-	(wire
-		(pts
-			(xy 153.67 55.88) (xy 170.18 55.88)
+			(xy 144.78 48.26) (xy 170.18 48.26)
+		)
+		(stroke
+			(width 0)
+			(type default)
+		)
+	)
+	(wire
+		(pts
+			(xy 144.78 55.88) (xy 170.18 55.88)
 		)
 		(stroke
@@
 		)
 	)
-	(label "uC_I2C1_SDA"
-		(at 156.21 48.26 0)
+	(label "5V_uC_I2C1_SDA"
+		(at 149.86 48.26 0)
 		(effects
 			(font
@@
 		)
 	)
-	(label "uC_I2C1_SCL"
-		(at 154.94 55.88 0)
+	(label "5V_uC_I2C1_SCL"
+		(at 149.86 55.88 0)
 		(effects
 			(font
@@
 		)
 	)
-	(hierarchical_label "uC_I2C1_SDA"
+	(hierarchical_label "5V_uC_I2C1_SDA"
 		(shape input)
-		(at 153.67 48.26 180)
+		(at 144.78 48.26 180)
 		(effects
 			(font
@@
 		)
 	)
-	(hierarchical_label "uC_I2C1_SCL"
+	(hierarchical_label "5V_uC_I2C1_SCL"
 		(shape input)
-		(at 153.67 55.88 180)
+		(at 144.78 55.88 180)
 		(effects
 			(font

Commit message: Rearranged Project
Rearranged project pages to have a block diagram and upper level collector for all future hierarchical pages to be collected under when adding power pages. Started on Power conversion with 12V input jack.
Parts:
- renumbered C16 to C22, C17 to C23, C18 to C24, R13 to R20, R12 to R21, U2 to U9
Changed lines of the file:
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@@
 		(dnp no)
 		(fields_autoplaced yes)
-		(property "Reference" "#PWR028"
+		(property "Reference" "#PWR037"
 			(at 69.85 100.33 0)
 			(hide yes)
@@
 		(instances
 			(project "openKVM-X01"
-				(path "/e7c0374d-64bc-4089-b9c4-51fd59a7a9a1/b7508bf7-0e2e-492c-8bf4-48d4e3c671b8"
-					(reference "#PWR028")
+				(path "/2ca004d4-d0d6-4c87-a313-b0e1d2005e00/93c519a5-1468-4f17-938e-a4b41050cbf5/b7508bf7-0e2e-492c-8bf4-48d4e3c671b8"
+					(reference "#PWR037")
 					(unit 1)
 				)
@@
 		(dnp no)
 		(fields_autoplaced yes)
-		(property "Reference" "C18"
+		(property "Reference" "C24"
 			(at 223.52 27.9399 0)
 			(show_name no)
@@
 		(instances
 			(project "openKVM-X01"
-				(path "/e7c0374d-64bc-4089-b9c4-51fd59a7a9a1/b7508bf7-0e2e-492c-8bf4-48d4e3c671b8"
-					(reference "C18")
+				(path "/2ca004d4-d0d6-4c87-a313-b0e1d2005e00/93c519a5-1468-4f17-938e-a4b41050cbf5/b7508bf7-0e2e-492c-8bf4-48d4e3c671b8"
+					(reference "C24")
 					(unit 1)
 				)
@@
 		(dnp no)
 		(fields_autoplaced yes)
-		(property "Reference" "R12"
+		(property "Reference" "R21"
 			(at 72.39 86.3599 0)
 			(show_name no)
@@
 		(instances
 			(project "openKVM-X01"
-				(path "/e7c0374d-64bc-4089-b9c4-51fd59a7a9a1/b7508bf7-0e2e-492c-8bf4-48d4e3c671b8"
-					(reference "R12")
+				(path "/2ca004d4-d0d6-4c87-a313-b0e1d2005e00/93c519a5-1468-4f17-938e-a4b41050cbf5/b7508bf7-0e2e-492c-8bf4-48d4e3c671b8"
+					(reference "R21")
 					(unit 1)
 				)
@@
 		(in_pos_files yes)
 		(dnp no)
-		(property "Reference" "U2"
+		(property "Reference" "U9"
 			(at 236.6167 40.64 0)
 			(show_name no)
@@
 		(instances
 			(project "openKVM-X01"
-				(path "/e7c0374d-64bc-4089-b9c4-51fd59a7a9a1/b7508bf7-0e2e-492c-8bf4-48d4e3c671b8"
-					(reference "U2")
+				(path "/2ca004d4-d0d6-4c87-a313-b0e1d2005e00/93c519a5-1468-4f17-938e-a4b41050cbf5/b7508bf7-0e2e-492c-8bf4-48d4e3c671b8"
+					(reference "U9")
 					(unit 1)
 				)
@@
 		(dnp no)
 		(fields_autoplaced yes)
-		(property "Reference" "R13"
+		(property "Reference" "R20"
 			(at 59.69 86.3599 0)
 			(show_name no)
@@
 		(instances
 			(project "openKVM-X01"
-				(path "/e7c0374d-64bc-4089-b9c4-51fd59a7a9a1/b7508bf7-0e2e-492c-8bf4-48d4e3c671b8"
-					(reference "R13")
+				(path "/2ca004d4-d0d6-4c87-a313-b0e1d2005e00/93c519a5-1468-4f17-938e-a4b41050cbf5/b7508bf7-0e2e-492c-8bf4-48d4e3c671b8"
+					(reference "R20")
 					(unit 1)
 				)
@@
 		(dnp no)
 		(fields_autoplaced yes)
-		(property "Reference" "#PWR029"
+		(property "Reference" "#PWR034"
 			(at 57.15 100.33 0)
 			(hide yes)
@@
 		(instances
 			(project "openKVM-X01"
-				(path "/e7c0374d-64bc-4089-b9c4-51fd59a7a9a1/b7508bf7-0e2e-492c-8bf4-48d4e3c671b8"
-					(reference "#PWR029")
+				(path "/2ca004d4-d0d6-4c87-a313-b0e1d2005e00/93c519a5-1468-4f17-938e-a4b41050cbf5/b7508bf7-0e2e-492c-8bf4-48d4e3c671b8"
+					(reference "#PWR034")
 					(unit 1)
 				)
@@
 		(dnp no)
 		(fields_autoplaced yes)
-		(property "Reference" "#PWR032"
+		(property "Reference" "#PWR035"
 			(at 68.58 24.13 0)
 			(hide yes)
@@
 		(instances
 			(project "openKVM-X01"
-				(path "/e7c0374d-64bc-4089-b9c4-51fd59a7a9a1/b7508bf7-0e2e-492c-8bf4-48d4e3c671b8"
-					(reference "#PWR032")
+				(path "/2ca004d4-d0d6-4c87-a313-b0e1d2005e00/93c519a5-1468-4f17-938e-a4b41050cbf5/b7508bf7-0e2e-492c-8bf4-48d4e3c671b8"
+					(reference "#PWR035")
 					(unit 1)
 				)
@@
 		(dnp no)
 		(fields_autoplaced yes)
-		(property "Reference" "#PWR035"
+		(property "Reference" "#PWR048"
 			(at 163.83 39.37 0)
 			(hide yes)
@@
 		(instances
 			(project "openKVM-X01"
-				(path "/e7c0374d-64bc-4089-b9c4-51fd59a7a9a1/b7508bf7-0e2e-492c-8bf4-48d4e3c671b8"
-					(reference "#PWR035")
+				(path "/2ca004d4-d0d6-4c87-a313-b0e1d2005e00/93c519a5-1468-4f17-938e-a4b41050cbf5/b7508bf7-0e2e-492c-8bf4-48d4e3c671b8"
+					(reference "#PWR048")
 					(unit 1)
 				)
@@
 		(instances
 			(project "openKVM-X01"
-				(path "/e7c0374d-64bc-4089-b9c4-51fd59a7a9a1/b7508bf7-0e2e-492c-8bf4-48d4e3c671b8"
+				(path "/2ca004d4-d0d6-4c87-a313-b0e1d2005e00/93c519a5-1468-4f17-938e-a4b41050cbf5/b7508bf7-0e2e-492c-8bf4-48d4e3c671b8"
 					(reference "U4")
 					(unit 1)
@@
 		(dnp no)
 		(fields_autoplaced yes)
-		(property "Reference" "#PWR033"
+		(property "Reference" "#PWR036"
 			(at 68.58 39.37 0)
 			(hide yes)
@@
 		(instances
 			(project "openKVM-X01"
-				(path "/e7c0374d-64bc-4089-b9c4-51fd59a7a9a1/b7508bf7-0e2e-492c-8bf4-48d4e3c671b8"
-					(reference "#PWR033")
+				(path "/2ca004d4-d0d6-4c87-a313-b0e1d2005e00/93c519a5-1468-4f17-938e-a4b41050cbf5/b7508bf7-0e2e-492c-8bf4-48d4e3c671b8"
+					(reference "#PWR036")
 					(unit 1)
 				)
@@
 		(dnp no)
 		(fields_autoplaced yes)
-		(property "Reference" "#PWR09"
+		(property "Reference" "#PWR049"
 			(at 182.88 96.52 0)
 			(hide yes)
@@
 		(instances
 			(project "openKVM-X01"
-				(path "/e7c0374d-64bc-4089-b9c4-51fd59a7a9a1/b7508bf7-0e2e-492c-8bf4-48d4e3c671b8"
-					(reference "#PWR09")
+				(path "/2ca004d4-d0d6-4c87-a313-b0e1d2005e00/93c519a5-1468-4f17-938e-a4b41050cbf5/b7508bf7-0e2e-492c-8bf4-48d4e3c671b8"
+					(reference "#PWR049")
 					(unit 1)
 				)
@@
 		(dnp no)
 		(fields_autoplaced yes)
-		(property "Reference" "#PWR037"
+		(property "Reference" "#PWR051"
 			(at 219.71 40.64 0)
 			(hide yes)
@@
 		(instances
 			(project "openKVM-X01"
-				(path "/e7c0374d-64bc-4089-b9c4-51fd59a7a9a1/b7508bf7-0e2e-492c-8bf4-48d4e3c671b8"
-					(reference "#PWR037")
+				(path "/2ca004d4-d0d6-4c87-a313-b0e1d2005e00/93c519a5-1468-4f17-938e-a4b41050cbf5/b7508bf7-0e2e-492c-8bf4-48d4e3c671b8"
+					(reference "#PWR051")
 					(unit 1)
 				)
@@
 		(dnp no)
 		(fields_autoplaced yes)
-		(property "Reference" "C17"
+		(property "Reference" "C23"
 			(at 167.64 26.6699 0)
 			(show_name no)
@@
 		(instances
 			(project "openKVM-X01"
-				(path "/e7c0374d-64bc-4089-b9c4-51fd59a7a9a1/b7508bf7-0e2e-492c-8bf4-48d4e3c671b8"
-					(reference "C17")
+				(path "/2ca004d4-d0d6-4c87-a313-b0e1d2005e00/93c519a5-1468-4f17-938e-a4b41050cbf5/b7508bf7-0e2e-492c-8bf4-48d4e3c671b8"
+					(reference "C23")
 					(unit 1)
 				)
@@
 		(dnp no)
 		(fields_autoplaced yes)
-		(property "Reference" "#PWR013"
+		(property "Reference" "#PWR052"
 			(at 238.76 68.58 0)
 			(hide yes)
@@
 		(instances
 			(project "openKVM-X01"
-				(path "/e7c0374d-64bc-4089-b9c4-51fd59a7a9a1/b7508bf7-0e2e-492c-8bf4-48d4e3c671b8"
-					(reference "#PWR013")
+				(path "/2ca004d4-d0d6-4c87-a313-b0e1d2005e00/93c519a5-1468-4f17-938e-a4b41050cbf5/b7508bf7-0e2e-492c-8bf4-48d4e3c671b8"
+					(reference "#PWR052")
 					(unit 1)
 				)
@@
 		(dnp no)
 		(fields_autoplaced yes)
-		(property "Reference" "#PWR036"
+		(property "Reference" "#PWR050"
 			(at 219.71 25.4 0)
 			(hide yes)
@@
 		(instances
 			(project "openKVM-X01"
-				(path "/e7c0374d-64bc-4089-b9c4-51fd59a7a9a1/b7508bf7-0e2e-492c-8bf4-48d4e3c671b8"
-					(reference "#PWR036")
+				(path "/2ca004d4-d0d6-4c87-a313-b0e1d2005e00/93c519a5-1468-4f17-938e-a4b41050cbf5/b7508bf7-0e2e-492c-8bf4-48d4e3c671b8"
+					(reference "#PWR050")
 					(unit 1)
 				)
@@
 		(dnp no)
 		(fields_autoplaced yes)
-		(property "Reference" "C16"
+		(property "Reference" "C22"
 			(at 72.39 26.6699 0)
 			(show_name no)
@@
 		(instances
 			(project "openKVM-X01"
-				(path "/e7c0374d-64bc-4089-b9c4-51fd59a7a9a1/b7508bf7-0e2e-492c-8bf4-48d4e3c671b8"
-					(reference "C16")
+				(path "/2ca004d4-d0d6-4c87-a313-b0e1d2005e00/93c519a5-1468-4f17-938e-a4b41050cbf5/b7508bf7-0e2e-492c-8bf4-48d4e3c671b8"
+					(reference "C22")
 					(unit 1)
 				)
@@
 		(instances
 			(project "openKVM-X01"
-				(path "/e7c0374d-64bc-4089-b9c4-51fd59a7a9a1/b7508bf7-0e2e-492c-8bf4-48d4e3c671b8"
+				(path "/2ca004d4-d0d6-4c87-a313-b0e1d2005e00/93c519a5-1468-4f17-938e-a4b41050cbf5/b7508bf7-0e2e-492c-8bf4-48d4e3c671b8"
 					(reference "U5")
 					(unit 1)
@@
 		(dnp no)
 		(fields_autoplaced yes)
-		(property "Reference" "#PWR03"
+		(property "Reference" "#PWR044"
 			(at 87.63 100.33 0)
 			(hide yes)
@@
 		(instances
 			(project "openKVM-X01"
-				(path "/e7c0374d-64bc-4089-b9c4-51fd59a7a9a1/b7508bf7-0e2e-492c-8bf4-48d4e3c671b8"
-					(reference "#PWR03")
+				(path "/2ca004d4-d0d6-4c87-a313-b0e1d2005e00/93c519a5-1468-4f17-938e-a4b41050cbf5/b7508bf7-0e2e-492c-8bf4-48d4e3c671b8"
+					(reference "#PWR044")
 					(unit 1)
 				)
@@
 		(dnp no)
 		(fields_autoplaced yes)
-		(property "Reference" "#PWR034"
+		(property "Reference" "#PWR047"
 			(at 163.83 24.13 0)
 			(hide yes)
@@
 		(instances
 			(project "openKVM-X01"
-				(path "/e7c0374d-64bc-4089-b9c4-51fd59a7a9a1/b7508bf7-0e2e-492c-8bf4-48d4e3c671b8"
-					(reference "#PWR034")
-					(unit 1)
-				)
+				(path "/2ca004d4-d0d6-4c87-a313-b0e1d2005e00/93c519a5-1468-4f17-938e-a4b41050cbf5/b7508bf7-0e2e-492c-8bf4-48d4e3c671b8"
+					(reference "#PWR047")
+					(unit 1)
+				)
