File: Power.kicad_sch (KiCad schematic)
At the start: 0 parts

Commit message: Rearranged Project
Rearranged project pages to have a block diagram and upper level collector for all future hierarchical pages to be collected under when adding power pages. Started on Power conversion with 12V input jack.
Parts:
- added C15, C16, C17: C, symbol Device:C
- added D4: D_TVS, symbol Device:D_TVS
- added D5: D_Schottky, symbol Device:D_Schottky
- added J1: PJ-102AH, Connector_BarrelJack:BarrelJack_CUI_PJ-102AH_Horizontal, symbol Connector:Barrel_Jack_Switch
- added L1, L2: L, symbol Device:L
- added R10, R12: R, Resistor_SMD:R_0603_1608Metric, symbol Device:R
- added R7: 10k, Resistor_SMD:R_0603_1608Metric, symbol Device:R
- added U2: TPS562242B, Package_TO_SOT_SMD:SOT-563, symbol OpenKVM_PowerSupplies:TPS56x24x
Connections:
- new net: C15.1, D4.1 (A1), J1.1, L1.1
- new net: C16.1, D5.2 (A), L1.2
- new net: L2.2, R10.1
- new net +12V: D5.1 (K), R7.1, U2.1 (VIN)
- new net GND: C15.2, C16.2, D4.2 (A2), J1.2, R12.2, U2.3 (GND)
- new net U2_BST: C17.1, U2.4 (BST)
- new net U2_EN: R7.2, U2.5 (EN)
- new net U2_FB: R10.2, R12.1, U2.6 (FB)
- new net U2_SW: C17.2, L2.1, U2.2 (SW)
Other:
- note added: "PART SOMEWHAT SMALLER THAN I INITIALLY BELIEVED BUT WOULD NOT BE TRICKY TO ASSEMBLE WITH HOT PLATE."
- title: (none) -> POWER
