File: hdmi_mux.kicad_sch (KiCad schematic)
At the start: 4 parts, among them U3 TS3DV642A0RUAR

Commit message: Created Branch and Made Changes
Fixed I2C going into Mux shorting the 3V3 side and 5V side due to nets being the same names. Added grounding to HDMI Out connector. Fixed footprint for TS3DV642A0RUAR to use KiCAD default library footprint with EasyEDA 3D model.
Parts:
- U3: footprint (none) -> Package_DFN_QFN:WQFN-42-1EP_3.5x9mm_P0.5mm_EP2.05x7.55mm_ThermalVias
Changed lines of the file:
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@@
 			)
 		)
-		(property "Footprint" ""
+		(property "Footprint" "Package_DFN_QFN:WQFN-42-1EP_3.5x9mm_P0.5mm_EP2.05x7.55mm_ThermalVias"
 			(at 146.05 95.25 0)
 			(hide yes)

Commit message: Rearranged Project
Rearranged project pages to have a block diagram and upper level collector for all future hierarchical pages to be collected under when adding power pages. Started on Power conversion with 12V input jack.
Parts:
- renumbered C15 to C18, R7 to R13, R10 to R19
Changed lines of the file:
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@@
 		(dnp no)
 		(fields_autoplaced yes)
-		(property "Reference" "R7"
+		(property "Reference" "R13"
 			(at 175.26 48.2599 0)
 			(show_name no)
@@
 		(instances
 			(project "openKVM-X01"
-				(path "/e7c0374d-64bc-4089-b9c4-51fd59a7a9a1/cfd16a7f-110b-4ed7-bcc6-fad01c2502ae"
-					(reference "R7")
+				(path "/2ca004d4-d0d6-4c87-a313-b0e1d2005e00/93c519a5-1468-4f17-938e-a4b41050cbf5/cfd16a7f-110b-4ed7-bcc6-fad01c2502ae"
+					(reference "R13")
 					(unit 1)
 				)
@@
 		(dnp no)
 		(fields_autoplaced yes)
-		(property "Reference" "#PWR026"
+		(property "Reference" "#PWR027"
 			(at 107.95 34.29 0)
 			(hide yes)
@@
 		(instances
 			(project "openKVM-X01"
-				(path "/e7c0374d-64bc-4089-b9c4-51fd59a7a9a1/cfd16a7f-110b-4ed7-bcc6-fad01c2502ae"
-					(reference "#PWR026")
+				(path "/2ca004d4-d0d6-4c87-a313-b0e1d2005e00/93c519a5-1468-4f17-938e-a4b41050cbf5/cfd16a7f-110b-4ed7-bcc6-fad01c2502ae"
+					(reference "#PWR027")
 					(unit 1)
 				)
@@
 		(dnp no)
 		(fields_autoplaced yes)
-		(property "Reference" "#PWR025"
+		(property "Reference" "#PWR033"
 			(at 186.69 148.59 0)
 			(hide yes)
@@
 		(instances
 			(project "openKVM-X01"
-				(path "/e7c0374d-64bc-4089-b9c4-51fd59a7a9a1/cfd16a7f-110b-4ed7-bcc6-fad01c2502ae"
-					(reference "#PWR025")
+				(path "/2ca004d4-d0d6-4c87-a313-b0e1d2005e00/93c519a5-1468-4f17-938e-a4b41050cbf5/cfd16a7f-110b-4ed7-bcc6-fad01c2502ae"
+					(reference "#PWR033")
 					(unit 1)
 				)
@@
 		(instances
 			(project "openKVM-X01"
-				(path "/e7c0374d-64bc-4089-b9c4-51fd59a7a9a1/cfd16a7f-110b-4ed7-bcc6-fad01c2502ae"
+				(path "/2ca004d4-d0d6-4c87-a313-b0e1d2005e00/93c519a5-1468-4f17-938e-a4b41050cbf5/cfd16a7f-110b-4ed7-bcc6-fad01c2502ae"
 					(reference "U3")
 					(unit 1)
@@
 		(dnp no)
 		(fields_autoplaced yes)
-		(property "Reference" "#PWR027"
+		(property "Reference" "#PWR028"
 			(at 107.95 49.53 0)
 			(hide yes)
@@
 		(instances
 			(project "openKVM-X01"
-				(path "/e7c0374d-64bc-4089-b9c4-51fd59a7a9a1/cfd16a7f-110b-4ed7-bcc6-fad01c2502ae"
-					(reference "#PWR027")
+				(path "/2ca004d4-d0d6-4c87-a313-b0e1d2005e00/93c519a5-1468-4f17-938e-a4b41050cbf5/cfd16a7f-110b-4ed7-bcc6-fad01c2502ae"
+					(reference "#PWR028")
 					(unit 1)
 				)
@@
 		(dnp no)
 		(fields_autoplaced yes)
-		(property "Reference" "#PWR024"
+		(property "Reference" "#PWR032"
 			(at 172.72 46.99 0)
 			(hide yes)
@@
 		(instances
 			(project "openKVM-X01"
-				(path "/e7c0374d-64bc-4089-b9c4-51fd59a7a9a1/cfd16a7f-110b-4ed7-bcc6-fad01c2502ae"
-					(reference "#PWR024")
+				(path "/2ca004d4-d0d6-4c87-a313-b0e1d2005e00/93c519a5-1468-4f17-938e-a4b41050cbf5/cfd16a7f-110b-4ed7-bcc6-fad01c2502ae"
+					(reference "#PWR032")
 					(unit 1)
 				)
@@
 		(dnp no)
 		(fields_autoplaced yes)
-		(property "Reference" "R10"
+		(property "Reference" "R19"
 			(at 189.23 73.6599 0)
 			(show_name no)
@@
 		(instances
 			(project "openKVM-X01"
-				(path "/e7c0374d-64bc-4089-b9c4-51fd59a7a9a1/cfd16a7f-110b-4ed7-bcc6-fad01c2502ae"
-					(reference "R10")
+				(path "/2ca004d4-d0d6-4c87-a313-b0e1d2005e00/93c519a5-1468-4f17-938e-a4b41050cbf5/cfd16a7f-110b-4ed7-bcc6-fad01c2502ae"
+					(reference "R19")
 					(unit 1)
 				)
@@
 		(dnp no)
 		(fields_autoplaced yes)
-		(property "Reference" "C15"
+		(property "Reference" "C18"
 			(at 111.76 34.2899 0)
 			(show_name no)
@@
 		(instances
 			(project "openKVM-X01"
-				(path "/e7c0374d-64bc-4089-b9c4-51fd59a7a9a1/cfd16a7f-110b-4ed7-bcc6-fad01c2502ae"
-					(reference "C15")
+				(path "/2ca004d4-d0d6-4c87-a313-b0e1d2005e00/93c519a5-1468-4f17-938e-a4b41050cbf5/cfd16a7f-110b-4ed7-bcc6-fad01c2502ae"
+					(reference "C18")
 					(unit 1)
 				)
@@
 		(dnp no)
 		(fields_autoplaced yes)
-		(property "Reference" "#PWR015"
+		(property "Reference" "#PWR029"
 			(at 119.38 148.59 0)
 			(hide yes)
@@
 		(instances
 			(project "openKVM-X01"
-				(path "/e7c0374d-64bc-4089-b9c4-51fd59a7a9a1/cfd16a7f-110b-4ed7-bcc6-fad01c2502ae"
-					(reference "#PWR015")
+				(path "/2ca004d4-d0d6-4c87-a313-b0e1d2005e00/93c519a5-1468-4f17-938e-a4b41050cbf5/cfd16a7f-110b-4ed7-bcc6-fad01c2502ae"
+					(reference "#PWR029")
 					(unit 1)
 				)
