File: openKVM-X01.kicad_sch (KiCad schematic)
At the start: 45 parts, among them J2 HDMI_A_1.4, J3 HDMI_A_1.4, SW1 SW_SPDT, SW2 COM1_SELECT, U1 STM32F411VETx, U6 TCA9517ADGK, U7 74HC74, U8 74HC7014, Y1 Crystal

Commit message: Created Branch and Made Changes
Fixed I2C going into Mux shorting the 3V3 side and 5V side due to nets being the same names. Added grounding to HDMI Out connector. Fixed footprint for TS3DV642A0RUAR to use KiCAD default library footprint with EasyEDA 3D model.
Connections:
- net GND: now also J3.11 (CKS), J3.17 (GND), J3.2 (D2S), J3.5 (D1S), J3.8 (D0S), J3.SH
- net EDID_EMULATION/uC_I2C1_SCL renamed EDID_EMULATION/5V_uC_I2C1_SCL
- net EDID_EMULATION/uC_I2C1_SDA renamed EDID_EMULATION/5V_uC_I2C1_SDA
Other:
- sheet EDID_EMULATION ports: added 5V_uC_I2C1_SCL, 5V_uC_I2C1_SDA; removed uC_I2C1_SCL, uC_I2C1_SDA
- moved on the sheet: J3
